File: lem-adapter-board/lem_comm.kicad_sch (KiCad schematic)
At the start: 9 parts, among them J1 Conn_01x04

Commit message: Changed order in lem adapter connector
Connections:
- net +15V: now also J1.4 (Pin_4); no longer J1.1 (Pin_1)
- net -15V: now also J1.3 (Pin_3); no longer J1.4 (Pin_4)
- net GND: now also J1.1 (Pin_1); no longer J1.3 (Pin_3)
Changed lines of the file:
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@@
   (junction (at 51.943 69.85) (diameter 0) (color 0 0 0 0)
   )
-  (wire (pts (xy 48.387 33.655) (xy 45.72 33.655))
-    (stroke (width 0) (type default) (color 0 0 0 0))
-  )
   (wire (pts (xy 35.814 59.69) (xy 35.814 60.833))
-    (stroke (width 0) (type default) (color 0 0 0 0))
-  )
-  (wire (pts (xy 48.387 36.195) (xy 48.387 40.513))
     (stroke (width 0) (type default) (color 0 0 0 0))
   )
@@
     (stroke (width 0) (type default) (color 0 0 0 0))
   )
+  (wire (pts (xy 45.847 33.655) (xy 48.387 33.655))
+    (stroke (width 0) (type default) (color 0 0 0 0))
+  )
   (wire (pts (xy 43.053 60.833) (xy 51.943 60.833))
+    (stroke (width 0) (type default) (color 0 0 0 0))
+  )
+  (wire (pts (xy 45.847 28.575) (xy 48.387 28.575))
     (stroke (width 0) (type default) (color 0 0 0 0))
   )
@@
     (stroke (width 0) (type default) (color 0 0 0 0))
   )
-  (wire (pts (xy 40.513 39.624) (xy 45.72 39.624))
-    (stroke (width 0) (type default) (color 0 0 0 0))
-  )
   (wire (pts (xy 51.943 60.833) (xy 59.182 60.833))
     (stroke (width 0) (type default) (color 0 0 0 0))
@@
     (stroke (width 0) (type default) (color 0 0 0 0))
   )
-  (wire (pts (xy 48.387 26.035) (xy 48.387 28.575))
-    (stroke (width 0) (type default) (color 0 0 0 0))
-  )
   (wire (pts (xy 43.053 69.85) (xy 35.814 69.85))
     (stroke (width 0) (type default) (color 0 0 0 0))
   )
-  (wire (pts (xy 45.72 33.655) (xy 45.72 39.624))
+  (wire (pts (xy 45.847 36.195) (xy 48.387 36.195))
+    (stroke (width 0) (type default) (color 0 0 0 0))
+  )
+  (wire (pts (xy 45.847 31.115) (xy 48.387 31.115))
     (stroke (width 0) (type default) (color 0 0 0 0))
   )
@@
   )
   (wire (pts (xy 35.814 60.833) (xy 35.814 62.23))
-    (stroke (width 0) (type default) (color 0 0 0 0))
-  )
-  (wire (pts (xy 40.513 31.115) (xy 48.387 31.115))
     (stroke (width 0) (type default) (color 0 0 0 0))
   )
@@
     (effects (font (size 1.27 1.27)) (justify left bottom))
   )
-  (label "-15V" (at 48.387 40.513 0)
-    (effects (font (size 1.27 1.27)) (justify left bottom))
+  (label "-15V" (at 45.847 33.655 180)
+    (effects (font (size 1.27 1.27)) (justify right bottom))
   )
   (label "-15V" (at 24.511 31.115 0)
@@
     (effects (font (size 1.27 1.27)) (justify right bottom))
   )
-  (label "+15V" (at 48.387 26.035 0)
-    (effects (font (size 1.27 1.27)) (justify left bottom))
+  (label "+15V" (at 45.847 36.195 180)
+    (effects (font (size 1.27 1.27)) (justify right bottom))
   )
   (label "Iout" (at 33.274 52.07 180)
@@
     (effects (font (size 1.27 1.27)) (justify left bottom))
   )
-  (label "GND" (at 40.513 39.624 180)
+  (label "GND" (at 45.847 28.575 180)
     (effects (font (size 1.27 1.27)) (justify right bottom))
   )
-  (label "Iout" (at 40.513 31.115 180)
+  (label "Iout" (at 45.847 31.115 180)
     (effects (font (size 1.27 1.27)) (justify right bottom))
   )
