File: analog-buffer-six-channels/analog-buffer-six-channels.kicad_pcb (KiCad board)
At the start: 2 copper layers, 32.1 x 35 mm, 31 parts, among them J1 Conn_02x10_Odd_Even, J2 Conn_02x08_Odd_Even, U1 Opamp_Dual, U2 Opamp_Dual, U3 Opamp_Dual

Commit message: Generated gerber files for analog-buffer board
Parts:
- added R14: DNP, Resistor_SMD:R_0805_2012Metric, B.Cu at (54.3, 60.8)
Routing:
- net -VCC: track 47.3 -> 49.5 mm
Changed lines of the file:
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@@
     (descr "Mounting Hole 3.2mm, no annular, M3")
     (tags "mounting hole 3.2mm no annular m3")
-    (attr exclude_from_pos_files exclude_from_bom)
+    (attr board_only exclude_from_pos_files exclude_from_bom)
     (fp_text reference "REF**" (at 0 -4.2) (layer "F.SilkS") hide
       (effects (font (size 1 1) (thickness 0.15)))
@@
     (fp_circle (center 0 0) (end 3.2 0) (layer "Cmts.User") (width 0.15) (fill none))
     (fp_circle (center 0 0) (end 3.45 0) (layer "F.CrtYd") (width 0.05) (fill none))
-    (pad "" np_thru_hole circle (at 0 0) (size 3.2 3.2) (drill 3.2) (layers *.Cu *.Mask))
+    (pad "" np_thru_hole circle locked (at 0 0) (size 3.2 3.2) (drill 3.2) (layers *.Cu *.Mask))
   )
   (footprint "Capacitor_SMD:C_0805_2012Metric" (layer "F.Cu")
@@
     )
   )
-  (footprint "MountingHole:MountingHole_3.2mm_M3" (layer "F.Cu")
+  (footprint "MountingHole:MountingHole_3.2mm_M3" locked (layer "F.Cu")
     (at 81.5086 64.77)
     (descr "Mounting Hole 3.2mm, no annular, M3")
     (tags "mounting hole 3.2mm no annular m3")
-    (attr exclude_from_pos_files exclude_from_bom)
+    (attr board_only exclude_from_pos_files exclude_from_bom)
     (fp_text reference "REF**" (at 0 -4.2) (layer "F.SilkS") hide
       (effects (font (size 1 1) (thickness 0.15)))
@@
     (fp_circle (center 0 0) (end 3.2 0) (layer "Cmts.User") (width 0.15) (fill none))
     (fp_circle (center 0 0) (end 3.45 0) (layer "F.CrtYd") (width 0.05) (fill none))
-    (pad "" np_thru_hole circle (at 0 0) (size 3.2 3.2) (drill 3.2) (layers *.Cu *.Mask))
+    (pad "" np_thru_hole circle locked (at 0 0) (size 3.2 3.2) (drill 3.2) (layers *.Cu *.Mask))
   )
   (footprint "LED_SMD:LED_0805_2012Metric_Pad1.15x1.40mm_HandSolder" (layer "F.Cu")
@@
   )
   (footprint "Resistor_SMD:R_0805_2012Metric" (layer "B.Cu")
+    (at 54.2798 60.7587 90)
+    (descr "Resistor SMD 0805 (2012 Metric), square (rectangular) end terminal, IPC_7351 nominal, (Body size source: IPC-SM-782 page 72, https://www.pcb-3d.com/wordpress/wp-content/uploads/ipc-sm-782a_amendment_1_and_2.pdf), generated with kicad-footprint-generator")
+    (tags "resistor")
+    (property "Sheetfile" "analog-buffer-six-channels.kicad_sch")
+    (property "Sheetname" "")
+    (attr smd)
+    (fp_text reference "R14" (at -2.3095 0 180) (layer "B.SilkS")
+      (effects (font (size 0.7 0.7) (thickness 0.15)) (justify mirror))
+    )
+    (fp_text value "DNP" (at 0 -1.65 90) (layer "B.Fab")
+      (effects (font (size 1 1) (thickness 0.15)) (justify mirror))
+    )
+    (fp_text user "${REFERENCE}" (at 0 0 90) (layer "B.Fab")
+      (effects (font (size 0.5 0.5) (thickness 0.08)) (justify mirror))
+    )
+    (fp_line (start -0.227064 -0.735) (end 0.227064 -0.735) (layer "B.SilkS") (width 0.12))
+    (fp_line (start -0.227064 0.735) (end 0.227064 0.735) (layer "B.SilkS") (width 0.12))
+    (fp_line (start 1.68 0.95) (end 1.68 -0.95) (layer "B.CrtYd") (width 0.05))
+    (fp_line (start 1.68 -0.95) (end -1.68 -0.95) (layer "B.CrtYd") (width 0.05))
+    (fp_line (start -1.68 -0.95) (end -1.68 0.95) (layer "B.CrtYd") (width 0.05))
+    (fp_line (start -1.68 0.95) (end 1.68 0.95) (layer "B.CrtYd") (width 0.05))
+    (fp_line (start 1 0.625) (end 1 -0.625) (layer "B.Fab") (width 0.1))
+    (fp_line (start 1 -0.625) (end -1 -0.625) (layer "B.Fab") (width 0.1))
+    (fp_line (start -1 -0.625) (end -1 0.625) (layer "B.Fab") (width 0.1))
+    (fp_line (start -1 0.625) (end 1 0.625) (layer "B.Fab") (width 0.1))
+    (pad "1" smd roundrect (at -0.9125 0 90) (size 1.025 1.4) (layers "B.Cu" "B.Paste" "B.Mask") (roundrect_rratio 0.243902)
+      (net 3 "-VCC") (pintype "passive"))
+    (pad "2" smd roundrect (at 0.9125 0 90) (size 1.025 1.4) (layers "B.Cu" "B.Paste" "B.Mask") (roundrect_rratio 0.243902)
+      (net 2 "GND") (pintype "passive"))
+    (model "${KICAD6_3DMODEL_DIR}/Resistor_SMD.3dshapes/R_0805_2012Metric.wrl"
+      (offset (xyz 0 0 0))
+      (scale (xyz 1 1 1))
+      (rotate (xyz 0 0 0))
+    )
+  )
+  (footprint "Resistor_SMD:R_0805_2012Metric" (layer "B.Cu")
     (at 66.6458 37.0728)
     (descr "Resistor SMD 0805 (2012 Metric), square (rectangular) end terminal, IPC_7351 nominal, (Body size source: IPC-SM-782 page 72, https://www.pcb-3d.com/wordpress/wp-content/uploads/ipc-sm-782a_amendment_1_and_2.pdf), generated with kicad-footprint-generator")
@@
   (via (at 66.2667 47.6362) (size 0.8) (drill 0.4) (layers "F.Cu" "B.Cu") (net 3))
   (segment (start 61.1886 52.8828) (end 60.8838 53.1876) (width 0.3) (layer "B.Cu") (net 3))
+  (segment (start 56.5185 61.6712) (end 56.5262 61.6789) (width 0.254) (layer "B.Cu") (net 3))
   (segment (start 60.0456 60.4012) (end 57.8039 60.4012) (width 0.3) (layer "B.Cu") (net 3))
+  (segment (start 54.2798 61.6712) (end 56.5185 61.6712) (width 0.254) (layer "B.Cu") (net 3))
   (segment (start 57.8039 60.4012) (end 56.5262 61.6789) (width 0.3) (layer "B.Cu") (net 3))
   (segment (start 60.8838 53.1876) (end 60.8838 59.563) (width 0.3) (layer "B.Cu") (net 3))
