File: adc-fiber-interface-board-six-channels/adc-fiber-interface-board-six-channels.kicad_sch (KiCad schematic)
At the start: 9 parts, among them J1 Conn_02x08_Odd_Even, U9 74HCT541

Commit message: Initial version of adc-fiber board
Connections:
- net RX1: now also U9.5 (A3); no longer U9.8 (A6)
- net RX1b: now also U9.15 (Y3); no longer U9.12 (Y6)
- net RX2: now also U9.6 (A4); no longer U9.9 (A7)
- net RX2b: now also U9.14 (Y4); no longer U9.11 (Y7)
- net TX4: now also U9.7 (A5); no longer U9.5 (A3)
- net TX4b: now also U9.13 (Y5); no longer U9.15 (Y3)
- net TX5: now also U9.8 (A6); no longer U9.6 (A4)
- net TX5b: now also U9.12 (Y6); no longer U9.14 (Y4)
- net TX6: now also U9.9 (A7); no longer U9.7 (A5)
- net TX6b: now also U9.11 (Y7); no longer U9.13 (Y5)

Commit message: Started working on optic transceiver
Other:
- note added: "[1] Vcc powers the buffer and the optic transmitter and receivers. Vcc can be selecting by placing the proper resistor."
- note removed: "[1] Vcc powers the reference generator and the amplifier circuit. Vcc can be selected by removing or shorting these resistor, according to the desired voltage."
Changed lines of the file:
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@@
     (effects (font (size 1.27 1.27)) (justify left bottom))
   )
-  (text "[1] Vcc powers the reference generator and the amplifier \ncircuit. Vcc can be selected by removing or shorting these\nresistor, according to the desired voltage."
+  (text "[1] Vcc powers the buffer and the optic transmitter and \nreceivers. Vcc can be selecting by placing the proper \nresistor."
     (at 15.24 89.662 0)
     (effects (font (size 1.27 1.27)) (justify left bottom))

Commit message: Generated gerber files for adc-fiber-interface board
Other:
- note added: "[1] Vcc powers the buffer, the optic transmitter and receivers. Vcc can be selecting by placing the proper resistor."
- note removed: "[1] Vcc powers the buffer and the optic transmitter and receivers. Vcc can be selecting by placing the proper resistor."
Changed lines of the file:
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@@
     (effects (font (size 1.27 1.27)) (justify left bottom))
   )
-  (text "[1] Vcc powers the buffer and the optic transmitter and \nreceivers. Vcc can be selecting by placing the proper \nresistor."
+  (text "[1] Vcc powers the buffer, the optic transmitter and \nreceivers. Vcc can be selecting by placing the proper \nresistor."
     (at 15.24 89.662 0)
     (effects (font (size 1.27 1.27)) (justify left bottom))
