File: optic-transceiver-board-2t6r/optic-transceiver-board-2t6r.kicad_sch (KiCad schematic)
At the start: 9 parts, among them J1 Conn_02x08_Odd_Even, U9 74HCT541

Commit message: Generated gerber files for optic-transceiver board
Other:
- note added: "[1] Vcc powers the buffer, the optic transmitter and receivers. Vcc can be selecting by placing the proper resistor."
- note removed: "[1] Vcc powers the buffer and the optic transmitter and receivers. Vcc can be selecting by placing the proper resistor."
Changed lines of the file:
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@@
     (effects (font (size 1.27 1.27)) (justify left bottom))
   )
-  (text "[1] Vcc powers the buffer and the optic transmitter and \nreceivers. Vcc can be selecting by placing the proper \nresistor."
+  (text "[1] Vcc powers the buffer, the optic transmitter and \nreceivers. Vcc can be selecting by placing the proper \nresistor."
     (at 225.044 94.361 0)
     (effects (font (size 1.27 1.27)) (justify left bottom))
