File: adc-board-six-channels/adc-board-six-channels.kicad_sch (KiCad schematic)
At the start: 8 parts, among them J1 Conn_02x08_Odd_Even, J2 Conn_02x08_Odd_Even

Commit message: Generated gerber for adc-board
Other:
- note added: "[1] Vcc powers the ADCs and it can be selected by removing or shorting these resistors, according to the desired voltage."
- note added: "[2]"
- note added: "[2] These resistor are supposed to avoid ringing on the CLK and CS lines due to the connectos being too long. They should be a small value or shorted."
- note removed: "[1] Vcc powers the reference generator and the amplifier circuit. Vcc can be selected by removing or shorting these resistor, according to the desired voltage."
Changed lines of the file:
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@@
     (stroke (width 0) (type default) (color 0 0 0 0))
   )
-  (text "[1] Vcc powers the reference generator and the amplifier \ncircuit. Vcc can be selected by removing or shorting these\nresistor, according to the desired voltage."
+  (text "[2]" (at 226.314 22.352 0)
+    (effects (font (size 1.27 1.27)) (justify left bottom))
+  )
+  (text "[2] These resistor are supposed to avoid ringing on the\nCLK and CS lines due to the connectos being too long.\nThey should be a small value or shorted."
+    (at 17.018 96.012 0)
+    (effects (font (size 1.27 1.27)) (justify left bottom))
+  )
+  (text "[1] Vcc powers the ADCs and it can be selected by removing \nor shorting these resistors, according to the desired voltage."
     (at 17.018 88.138 0)
     (effects (font (size 1.27 1.27)) (justify left bottom))
