File: amplifier-board-six-channels/sigcond.kicad_sch (KiCad schematic)
At the start: 14 parts, among them U1 Opamp_Dual

Commit message: Generated gerber files for amplifier board
Other:
- note added: "[1]"
- note added: "[1] These resistors should form a voltage divider on the reference voltage. They are intended to give different offset levels for each channel. If the reference voltage should be exactly the one from the reference generator, then the lower resistor and the 100 nF capacitor should be removed, while the upper resistor should be shorted. Do not remove the lower resistor while leaving the capacitor, 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"
- note added: "[2] If S_in is a current signal, the resistor between S_in and ground must be placed. In this case, the additional series resistor at the inverting input of the amplifier could also be placed to compensate for the gain mismatch. If S_in is a voltage signal, the resistor between S_in and ground should not be placed, and the series resistor on the amplifier's inverting input should be shorted."
- note added: "[3]"
- note added: "[3] This resistor and this capacitor could form a low-pass filter at the amplifier's output. Additionally, the capacitor could be removed and the resistor placed, in order to damp oscillations at the amplifiers output due to capacitive behavior of the output connectors."
Changed lines of the file:
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@@
     (stroke (width 0) (type default) (color 0 0 0 0))
+  )
+  (text "[2]" (at 22.987 87.249 0)
+    (effects (font (size 1.27 1.27)) (justify left bottom))
+  )
+  (text "[3]" (at 60.452 90.678 0)
+    (effects (font (size 1.27 1.27)) (justify left bottom))
+  )
+  (text "[3] This resistor and this capacitor could form a low-pass\nfilter at the amplifier's output. Additionally, the capacitor\ncould be removed and the resistor placed, in order to damp \noscillations at the amplifiers output due to capacitive \nbehavior of the output connectors."
+    (at 117.729 58.039 0)
+    (effects (font (size 1.27 1.27)) (justify left bottom))
   )
   (text "[2]" (at 42.418 107.696 0)
     (effects (font (size 1.27 1.27)) (justify left bottom))
   )
+  (text "[1]" (at 21.717 53.086 0)
+    (effects (font (size 1.27 1.27)) (justify left bottom))
+  )
+  (text "[1] These resistors should form a voltage divider on the\nreference voltage. They are intended to give different \noffset levels for each channel. If the reference voltage\nshould be exactly the one from the reference generator, then\nthe lower resistor and the 100 nF capacitor should be removed,\nwhile the upper resistor should be shorted. Do not remove \nthe lower resistor while leaving the capacitor, as this \ncould be a large capacitive load for the reference generator."
+    (at 118.11 30.607 0)
+    (effects (font (size 1.27 1.27)) (justify left bottom))
+  )
+  (text "[2] If S_in is a current signal, the resistor between S_in\nand ground must be placed. In this case, the additional\nseries resistor at the inverting input of the amplifier could\nalso be placed to compensate for the gain mismatch. If S_in\nis a voltage signal, the resistor between S_in and ground should\nnot be placed, and the series resistor on the amplifier's\ninverting input should be shorted."
+    (at 118.237 46.228 0)
+    (effects (font (size 1.27 1.27)) (justify left bottom))
+  )

Commit message: Updated gain values and created bom for amplifier board
Parts:
- R3, R7: value TBD -> 22k
Changed lines of the file:
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@@
       (effects (font (size 1.27 1.27)) (justify left))
     )
-    (property "Value" "TBD" (id 1) (at 50.038 93.98 90)
+    (property "Value" "22k" (id 1) (at 50.038 93.98 90)
       (effects (font (size 1.27 1.27)) (justify left))
     )
@@
       (effects (font (size 1.27 1.27)) (justify left))
     )
-    (property "Value" "TBD" (id 1) (at 41.91 78.74 0)
-      (effects (font (size 1.27 1.27)) (justify left))
-    )
+    (property "Value" "22k" (id 1) (at 41.91 78.74 0)
+      (effects (font (size 1.27 1.27)) (justify left))
+    )
