File: digital-isolator-2t6r/adum241x.kicad_sch (KiCad schematic)
At the start: 13 parts

Commit message: Added copper tracks to digital iso 2t6r board for in-house fab
Parts:
- C1, C3: value (none) -> 1uF; footprint (none) -> Capacitor_SMD:C_0805_2012Metric_Pad1.18x1.45mm_HandSolder
- C2, C4: value (none) -> 100nF; footprint (none) -> Capacitor_SMD:C_0805_2012Metric_Pad1.18x1.45mm_HandSolder
- R1, R2, R3, R4: value (none) -> 47R; footprint (none) -> Resistor_SMD:R_0805_2012Metric_Pad1.20x1.40mm_HandSolder
- U1: value (none) -> ADuM1401xRW; footprint (none) -> Package_SO:SOIC-16W_7.5x10.3mm_P1.27mm
Changed lines of the file:
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@@
       (effects (font (size 1.27 1.27)) (justify left))
     )
-    (property "Value" "" (id 1) (at 83.566 23.114 0)
+    (property "Value" "1uF" (id 1) (at 83.566 23.114 0)
       (effects (font (size 1.27 1.27)) (justify left))
     )
-    (property "Footprint" "" (id 2) (at 81.788 21.844 0)
+    (property "Footprint" "Capacitor_SMD:C_0805_2012Metric_Pad1.18x1.45mm_HandSolder" (id 2) (at 81.788 21.844 0)
       (effects (font (size 1.27 1.27)) hide)
     )
@@
       (effects (font (size 1.27 1.27)) (justify left))
     )
-    (property "Value" "" (id 1) (at 165.862 23.114 0)
+    (property "Value" "1uF" (id 1) (at 165.862 23.114 0)
       (effects (font (size 1.27 1.27)) (justify left))
     )
-    (property "Footprint" "" (id 2) (at 164.084 21.844 0)
+    (property "Footprint" "Capacitor_SMD:C_0805_2012Metric_Pad1.18x1.45mm_HandSolder" (id 2) (at 164.084 21.844 0)
       (effects (font (size 1.27 1.27)) hide)
     )
@@
     (in_bom yes) (on_board yes)
     (property "Reference" "R1" (id 0) (at 166.624 32.766 90))
-    (property "Value" "" (id 1) (at 166.624 36.576 90))
-    (property "Footprint" "" (id 2) (at 166.624 34.544 0)
+    (property "Value" "47R" (id 1) (at 166.624 36.576 90))
+    (property "Footprint" "Resistor_SMD:R_0805_2012Metric_Pad1.20x1.40mm_HandSolder" (id 2) (at 166.624 34.544 0)
       (effects (font (size 1.27 1.27)) hide)
     )
@@
     (in_bom yes) (on_board yes) (fields_autoplaced)
     (property "Reference" "U1" (id 0) (at 124.206 17.272 0))
-    (property "Value" "" (id 1) (at 124.206 19.812 0))
-    (property "Footprint" "" (id 2) (at 124.206 52.197 0)
+    (property "Value" "ADuM1401xRW" (id 1) (at 124.206 19.812 0))
+    (property "Footprint" "Package_SO:SOIC-16W_7.5x10.3mm_P1.27mm" (id 2) (at 124.206 52.197 0)
       (effects (font (size 1.27 1.27)) hide)
     )
@@
     (in_bom yes) (on_board yes)
     (property "Reference" "R2" (id 0) (at 77.724 35.306 90))
-    (property "Value" "" (id 1) (at 77.724 38.862 90))
-    (property "Footprint" "" (id 2) (at 77.724 37.084 0)
+    (property "Value" "47R" (id 1) (at 77.724 38.862 90))
+    (property "Footprint" "Resistor_SMD:R_0805_2012Metric_Pad1.20x1.40mm_HandSolder" (id 2) (at 77.724 37.084 0)
       (effects (font (size 1.27 1.27)) hide)
     )
@@
       (effects (font (size 1.27 1.27)) (justify left))
     )
-    (property "Value" "" (id 1) (at 173.482 23.114 0)
+    (property "Value" "100nF" (id 1) (at 173.482 23.114 0)
       (effects (font (size 1.27 1.27)) (justify left))
     )
-    (property "Footprint" "" (id 2) (at 171.704 21.844 0)
+    (property "Footprint" "Capacitor_SMD:C_0805_2012Metric_Pad1.18x1.45mm_HandSolder" (id 2) (at 171.704 21.844 0)
       (effects (font (size 1.27 1.27)) hide)
     )
@@
     (in_bom yes) (on_board yes)
     (property "Reference" "R4" (id 0) (at 166.624 45.974 90))
-    (property "Value" "" (id 1) (at 166.624 49.784 90))
-    (property "Footprint" "" (id 2) (at 166.624 47.752 0)
+    (property "Value" "47R" (id 1) (at 166.624 49.784 90))
+    (property "Footprint" "Resistor_SMD:R_0805_2012Metric_Pad1.20x1.40mm_HandSolder" (id 2) (at 166.624 47.752 0)
       (effects (font (size 1.27 1.27)) hide)
     )
@@
     (in_bom yes) (on_board yes)
     (property "Reference" "R3" (id 0) (at 166.624 39.624 90))
-    (property "Value" "" (id 1) (at 166.624 43.434 90))
-    (property "Footprint" "" (id 2) (at 166.624 41.402 0)
+    (property "Value" "47R" (id 1) (at 166.624 43.434 90))
+    (property "Footprint" "Resistor_SMD:R_0805_2012Metric_Pad1.20x1.40mm_HandSolder" (id 2) (at 166.624 41.402 0)
       (effects (font (size 1.27 1.27)) hide)
     )
@@
       (effects (font (size 1.27 1.27)) (justify left))
     )
-    (property "Value" "" (id 1) (at 91.186 23.114 0)
+    (property "Value" "100nF" (id 1) (at 91.186 23.114 0)
       (effects (font (size 1.27 1.27)) (justify left))
     )
-    (property "Footprint" "" (id 2) (at 89.408 21.844 0)
+    (property "Footprint" "Capacitor_SMD:C_0805_2012Metric_Pad1.18x1.45mm_HandSolder" (id 2) (at 89.408 21.844 0)
       (effects (font (size 1.27 1.27)) hide)
     )

Commit message: Added pull up resistor to digital isolator 2t6r board
Parts:
- added R17, R18: 100k, Resistor_SMD:R_0805_2012Metric_Pad1.20x1.40mm_HandSolder, symbol Device:R_Small
Connections:
- net VDDA: now also R17.2
- net VDDB: now also R18.1
- net at U1.10 (VE2): now also R18.2
- net at U1.7 (VE1): now also R17.1
- no-connect marks 2 -> 0
Changed lines of the file:
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@@
   (junction (at 164.084 24.892) (diameter 0) (color 0 0 0 0)
   )
-  (no_connect (at 108.966 42.672))
-  (no_connect (at 139.446 42.672))
   (wire (pts (xy 70.104 55.626) (xy 72.644 55.626))
     (stroke (width 0) (type default) (color 0 0 0 0))
@@
     (stroke (width 0) (type default) (color 0 0 0 0))
   )
+  (wire (pts (xy 147.066 42.672) (xy 149.606 42.672))
+    (stroke (width 0) (type default) (color 0 0 0 0))
+  )
   (wire (pts (xy 72.644 45.466) (xy 72.644 48.006))
     (stroke (width 0) (type default) (color 0 0 0 0))
@@
     (stroke (width 0) (type default) (color 0 0 0 0))
   )
+  (wire (pts (xy 98.806 42.672) (xy 101.346 42.672))
+    (stroke (width 0) (type default) (color 0 0 0 0))
+  )
   (wire (pts (xy 46.228 29.718) (xy 48.768 29.718))
     (stroke (width 0) (type default) (color 0 0 0 0))
@@
     (stroke (width 0) (type default) (color 0 0 0 0))
   )
+  (wire (pts (xy 139.446 42.672) (xy 141.986 42.672))
+    (stroke (width 0) (type default) (color 0 0 0 0))
+  )
   (wire (pts (xy 81.788 24.384) (xy 81.788 24.892))
     (stroke (width 0) (type default) (color 0 0 0 0))
@@
   )
   (wire (pts (xy 89.408 18.796) (xy 81.788 18.796))
+    (stroke (width 0) (type default) (color 0 0 0 0))
+  )
+  (wire (pts (xy 106.426 42.672) (xy 108.966 42.672))
     (stroke (width 0) (type default) (color 0 0 0 0))
   )
@@
     (effects (font (size 1.27 1.27)) (justify right bottom))
   )
+  (label "VDDB" (at 149.606 42.672 0)
+    (effects (font (size 1.27 1.27)) (justify left bottom))
+  )
   (label "GNDB" (at 141.986 47.752 0)
     (effects (font (size 1.27 1.27)) (justify left bottom))
@@
   (label "RX1_B" (at 48.768 29.718 0)
     (effects (font (size 1.27 1.27)) (justify left bottom))
+  )
+  (label "VDDA" (at 98.806 42.672 180)
+    (effects (font (size 1.27 1.27)) (justify right bottom))
   )
   (label "TX1_A'" (at 82.804 37.084 0)
@@
     (pin "2")
   )
+  (symbol (lib_id "Device:R_Small") (at 103.886 42.672 270) (unit 1)
+    (in_bom yes) (on_board yes)
+    (property "Reference" "R17" (id 0) (at 103.886 40.894 90))
+    (property "Value" "100k" (id 1) (at 103.886 44.45 90))
+    (property "Footprint" "Resistor_SMD:R_0805_2012Metric_Pad1.20x1.40mm_HandSolder" (id 2) (at 103.886 42.672 0)
+      (effects (font (size 1.27 1.27)) hide)
+    )
+    (property "Datasheet" "~" (id 3) (at 103.886 42.672 0)
+      (effects (font (size 1.27 1.27)) hide)
+    )
+    (pin "1")
+    (pin "2")
+  )
   (symbol (lib_id "Device:C_Small") (at 171.704 21.844 0) (unit 1)
     (in_bom yes) (on_board yes)
@@
       (effects (font (size 1.27 1.27)) hide)
     )
+    (pin "1")
+    (pin "2")
+  )
+  (symbol (lib_id "Device:R_Small") (at 144.526 42.672 270) (unit 1)
+    (in_bom yes) (on_board yes)
+    (property "Reference" "R18" (id 0) (at 144.526 40.894 90))
+    (property "Value" "100k" (id 1) (at 144.526 44.45 90))
+    (property "Footprint" "Resistor_SMD:R_0805_2012Metric_Pad1.20x1.40mm_HandSolder" (id 2) (at 144.526 42.672 0)
+      (effects (font (size 1.27 1.27)) hide)
+    )
+    (property "Datasheet" "~" (id 3) (at 144.526 42.672 0)
+      (effects (font (size 1.27 1.27)) hide)
+    )
