File: digital-isolator-6t2r/adum241x.kicad_sch (KiCad schematic)
At the start: 13 parts, among them U2 ADuM1401xRW

Commit message: Added pull up resistors to dig iso 6t2r board
Parts:
- added R19, R20: 100k, Resistor_SMD:R_0805_2012Metric_Pad1.20x1.40mm_HandSolder, symbol Device:R_Small
Connections:
- net VDDA: now also R19.2
- net VDDB: now also R20.1
- net at U2.10 (VE2): now also R20.2
- net at U2.7 (VE1): now also R19.1
- no-connect marks 2 -> 0
Changed lines of the file:
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@@
   (junction (at 164.084 24.892) (diameter 0) (color 0 0 0 0)
   )
-  (no_connect (at 108.966 42.672))
-  (no_connect (at 139.446 42.672))
   (wire (pts (xy 70.104 55.626) (xy 72.644 55.626))
     (stroke (width 0) (type default) (color 0 0 0 0))
@@
     (stroke (width 0) (type default) (color 0 0 0 0))
   )
+  (wire (pts (xy 139.446 42.672) (xy 141.986 42.672))
+    (stroke (width 0) (type default) (color 0 0 0 0))
+  )
   (wire (pts (xy 171.704 24.892) (xy 164.084 24.892))
     (stroke (width 0) (type default) (color 0 0 0 0))
@@
     (stroke (width 0) (type default) (color 0 0 0 0))
   )
+  (wire (pts (xy 147.066 42.672) (xy 149.606 42.672))
+    (stroke (width 0) (type default) (color 0 0 0 0))
+  )
   (wire (pts (xy 46.228 22.098) (xy 48.768 22.098))
     (stroke (width 0) (type default) (color 0 0 0 0))
@@
     (stroke (width 0) (type default) (color 0 0 0 0))
   )
+  (wire (pts (xy 106.426 42.672) (xy 108.966 42.672))
+    (stroke (width 0) (type default) (color 0 0 0 0))
+  )
   (wire (pts (xy 81.788 18.796) (xy 81.788 19.304))
     (stroke (width 0) (type default) (color 0 0 0 0))
@@
   )
   (wire (pts (xy 46.228 27.178) (xy 48.768 27.178))
+    (stroke (width 0) (type default) (color 0 0 0 0))
+  )
+  (wire (pts (xy 98.806 42.672) (xy 101.346 42.672))
     (stroke (width 0) (type default) (color 0 0 0 0))
   )
@@
     (effects (font (size 1.27 1.27)) (justify left bottom))
   )
+  (label "VDDA" (at 98.806 42.672 180)
+    (effects (font (size 1.27 1.27)) (justify right bottom))
+  )
   (label "VDDB" (at 141.986 24.892 0)
     (effects (font (size 1.27 1.27)) (justify left bottom))
@@
   (label "TX3_B'" (at 161.544 47.752 180)
     (effects (font (size 1.27 1.27)) (justify right bottom))
+  )
+  (label "VDDB" (at 149.606 42.672 0)
+    (effects (font (size 1.27 1.27)) (justify left bottom))
   )
   (label "TX1_A'" (at 106.426 37.592 180)
@@
     (pin "2")
   )
+  (symbol (lib_id "Device:R_Small") (at 144.526 42.672 270) (unit 1)
+    (in_bom yes) (on_board yes)
+    (property "Reference" "R20" (id 0) (at 144.526 40.894 90))
+    (property "Value" "100k" (id 1) (at 144.526 44.45 90))
+    (property "Footprint" "Resistor_SMD:R_0805_2012Metric_Pad1.20x1.40mm_HandSolder" (id 2) (at 144.526 42.672 0)
+      (effects (font (size 1.27 1.27)) hide)
+    )
+    (property "Datasheet" "~" (id 3) (at 144.526 42.672 0)
+      (effects (font (size 1.27 1.27)) hide)
+    )
+    (pin "1")
+    (pin "2")
+  )
   (symbol (lib_id "Device:R_Small") (at 166.624 41.402 90) (unit 1)
     (in_bom yes) (on_board yes)
@@
       (effects (font (size 1.27 1.27)) hide)
     )
+    (pin "1")
+    (pin "2")
+  )
+  (symbol (lib_id "Device:R_Small") (at 103.886 42.672 270) (unit 1)
+    (in_bom yes) (on_board yes)
+    (property "Reference" "R19" (id 0) (at 103.886 40.894 90))
+    (property "Value" "100k" (id 1) (at 103.886 44.45 90))
+    (property "Footprint" "Resistor_SMD:R_0805_2012Metric_Pad1.20x1.40mm_HandSolder" (id 2) (at 103.886 42.672 0)
+      (effects (font (size 1.27 1.27)) hide)
+    )
+    (property "Datasheet" "~" (id 3) (at 103.886 42.672 0)
+      (effects (font (size 1.27 1.27)) hide)
+    )
