File: digital-isolator-6t2r/digital-isolator-6t2r.kicad_pcb (KiCad board)
At the start: 2 copper layers, 47.1 x 42 mm, 34 parts, among them J1 Conn_02x08_Odd_Even, J2 Conn_02x08_Odd_Even, U1 ADuM1401xRW, U2 ADuM1401xRW

Commit message: Adapted pcb and generated gerbers for jlcpcb for dig iso 6t2r
Parts:
- R14, R17, R18, R19, R20, R6, R8: moved to F.Cu
- moved R19 8.04 mm to (106.0, 33.7), turned to 180 degrees
- moved R6 5.48 mm to (112.6, 58.1), turned to -90 degrees
- moved R14 4.38 mm to (110.8, 42.9)
- moved R15 4.17 mm to (113.2, 41.1), turned to -90 degrees
- moved R7 2.70 mm to (112.9, 53.2)
- moved R13 2.60 mm to (110.8, 46.8)
- moved R17 2.53 mm to (105.5, 53.5), turned to 180 degrees
- moved R10 2.53 mm to (109.2, 38.0), turned to 0 degrees
- moved R18 2.49 mm to (94.1, 53.7), turned to 180 degrees
- moved R8 2.47 mm to (90.2, 52.6), turned to 90 degrees
- moved R5 0.95 mm to (109.0, 63.3)
- moved R2 0.78 mm to (108.6, 54.8)
Routing:
- net VDDA: track 93.7 -> 101.9 mm, vias 1 -> 2
- net Net-(R19-Pad1): track 12.6 -> 6.01 mm, vias 1 -> 0
- net GNDA: track 2.72 -> 0.00 mm, vias 6 -> 17
- net /TX1_A: track 18.9 -> 16.6 mm
- net /adum241x/TX1_A': track 6.11 -> 4.32 mm
- net VDDB: track 95.2 -> 93.7 mm, vias 1 -> 2
- net /RX1_A: track 13.4 -> 14.5 mm
- net /RX4_A: track 15.4 -> 15.9 mm
- net /RX2_B: track 19.8 -> 20.3 mm, vias 1 -> 0
- net Net-(R18-Pad2): track 5.25 -> 5.01 mm, vias 1 -> 0
- net Net-(R17-Pad1): track 5.27 -> 5.33 mm, vias 1 -> 0
- net /RX5_A: track 14.9 -> 14.8 mm, vias 1 -> 0
- net /RX2_A: vias 1 -> 0
- net Net-(R20-Pad2): vias 1 -> 0
- net GNDB: vias 6 -> 11
Other:
- board text added: "GNDA"
- board text added: "GNDB"
- board text added: "RX1A"
- board text added: "RX1B"
- board text added: "RX2A"
- board text added: "RX2B"
- board text added: "RX3A"
- board text added: "RX4A"
- board text added: "RX5A"
- board text added: "RX6A"
- board text added: "TX1A"
- board text added: "TX1B"
- board text added: "TX2A"
- board text added: "TX2B"
- board text added: "TX3B"
- board text added: "TX4B"
- board text added: "TX5B"
- board text added: "TX6B"
- board text added: "VDDA"
- board text added: "VDDB"
- board text removed: "GND_A"
- board text removed: "GND_B"
- board text removed: "RX1_A"
- board text removed: "RX1_B"
- board text removed: "RX2_A"
- board text removed: "RX2_B"
- board text removed: "RX3_A"
- board text removed: "RX4_A"
- board text removed: "RX5_A"
- board text removed: "RX6_A"
- board text removed: "TX1_A"
- board text removed: "TX1_B"
- board text removed: "TX2_A"
- board text removed: "TX2_B"
- board text removed: "TX3_B"
- board text removed: "TX4_B"
- board text removed: "TX5_B"
- board text removed: "TX6_B"
- board text removed: "VDD_A"
- board text removed: "VDD_B"
