File: current-sensor-acs712/current-sensor-acs712.kicad_sch (KiCad schematic)
At the start: 19 parts

Commit message: Finished schematics for acs board, started pcb
Parts:
- added D1, D2: LED_Small_Filled, LED_SMD:LED_0805_2012Metric_Pad1.15x1.40mm_HandSolder, symbol Device:LED_Small_Filled
- added H1, H2: MountingHole, MountingHole:MountingHole_3.2mm_M3, symbol Mechanical:MountingHole
- added J1, J2: Conn_01x02, TerminalBlock_Phoenix:TerminalBlock_Phoenix_MKDS-1,5-2-5.08_1x02_P5.08mm_Horizontal, symbol Connector_Generic:Conn_01x02
- added J3: Conn_01x08, Connector_PinHeader_2.54mm:PinHeader_1x08_P2.54mm_Vertical, symbol Connector_Generic:Conn_01x08
- added R10, R8: DNP, Resistor_SMD:R_0805_2012Metric_Pad1.20x1.40mm_HandSolder, symbol Device:R_Small
- added R11, R12: 1k, Resistor_SMD:R_0805_2012Metric_Pad1.20x1.40mm_HandSolder, symbol Device:R_Small
- added R9: 0R, Resistor_SMD:R_0805_2012Metric_Pad1.20x1.40mm_HandSolder, symbol Device:R_Small
- gave numbers to parts that had none: 17
Connections:
- net GND: now also J3.5 (Pin_5), J3.6 (Pin_6), J3.7 (Pin_7), J3.8 (Pin_8), R11.2, R12.2
- net I_sens: now also J3.3 (Pin_3), R10.1, R9.1; no longer C8.1, R7.1
- net I_sens_filt: now also J3.4 (Pin_4)
- net VCC: now also D1.2 (A), J3.2 (Pin_2), R8.1; no longer R1.2
- net VDD: now also R1.2, D2.2 (A), J3.1 (Pin_1), R8.2
- net Vio: now also R10.2
- net Iio+ renamed I+
- net I+: now also J1.1 (Pin_1), J1.2 (Pin_2)
- net Iio- renamed I-
- net I-: now also J2.1 (Pin_1), J2.2 (Pin_2)
- new net: D1.1 (K), R11.1
- new net: D2.1 (K), R12.1
- new net Vio_amp: C8.1, R7.1, R9.2
Other:
- note added: "[5]"
- note added: "[6]"
- moved on the sheet: C4, C5, C6, C7, C8, R4, R5, R6, R7, U2A, U2B, U2C
