File: current-sensor-acs712/current-sensor-acs712.kicad_pcb (KiCad board)
At the start: 2 copper layers, 29 parts, among them J1 Conn_01x02, J2 Conn_01x02, J3 Conn_01x08, U1 ACS712xLCTR-20A, U2 Opamp_Dual

Commit message: Finishing acs712 board
Parts:
- R11, R12: moved to F.Cu
- R8: moved to B.Cu
- moved R11 4.78 mm to (104.8, 43.8), turned to 90 degrees
- moved H2 4.31 mm to (88.5, 67.3)
- moved D1 2.95 mm to (106.9, 43.8), turned to 90 degrees
- moved D2 2.44 mm to (111.6, 43.7), turned to 90 degrees
- moved H1 0.98 mm to (88.5, 44.8)
- moved R8 0.85 mm to (112.0, 47.5)
- moved R12 0.48 mm to (109.5, 43.8), turned to 90 degrees
- moved R9 0.44 mm to (102.0, 47.7)
- moved R10 0.44 mm to (99.9, 47.7)
- moved J3 0.15 mm to (115.0, 47.3)
Routing:
- net VDD: track 52.6 -> 59.9 mm
- net GND: track 0.00 -> 5.54 mm, vias 0 -> 6
- net VCC: track 22.7 -> 25.4 mm, vias 1 -> 2
- net /I-: track 0.00 -> 2.31 mm, vias 0 -> 3
- net Net-(D2-Pad1): track 0.00 -> 2.11 mm, vias 1 -> 0
- net Net-(D1-Pad1): track 0.00 -> 2.10 mm, vias 1 -> 0
- net /I+: track 0.00 -> 2.09 mm, vias 0 -> 3
- added copper zone on B.Cu, net /I-
- added copper zone on F.Cu, net /I-
- added copper zone on B.Cu, net GND
- added copper zone on F.Cu, net GND
Other:
- board outline added: 45 x 30 mm

Commit message: Finished acs pcb
Other:
- board text added: "Current sensor ACS board v0.1"
- board text added: "GND"
- board text added: "I+"
- board text added: "I-"
- board text added: "Is"
- board text added: "Isf"
- board text added: "Vcc"
- board text added: "Vdd"
Changed lines of the file:
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@@
     (property "Sheetname" "")
     (attr smd)
-    (fp_text reference "R5" (at -2.55 -0.025 unlocked) (layer "F.SilkS")
+    (fp_text reference "R5" (at -2.58 -1.03 unlocked) (layer "F.SilkS")
       (effects (font (size 0.7 0.7) (thickness 0.15)))
     )
@@
     (property "Sheetname" "")
     (attr through_hole)
-    (fp_text reference "J2" (at -3.45 3.825 180) (layer "F.SilkS")
+    (fp_text reference "J2" (at -3.69 4.05 180) (layer "F.SilkS")
       (effects (font (size 0.7 0.7) (thickness 0.15)))
     )
@@
     (property "Sheetname" "")
     (attr smd)
-    (fp_text reference "R12" (at -2.465 -0.01 unlocked) (layer "F.SilkS")
+    (fp_text reference "R12" (at 0.17 4.46 unlocked) (layer "F.SilkS")
       (effects (font (size 0.7 0.7) (thickness 0.15)))
     )
@@
     (property "Sheetname" "")
     (attr smd)
-    (fp_text reference "C7" (at -2.5875 2.05 unlocked) (layer "F.SilkS")
+    (fp_text reference "C7" (at -2.5525 1.81 unlocked) (layer "F.SilkS")
       (effects (font (size 0.7 0.7) (thickness 0.15)))
     )
@@
   )
   (footprint "Connector_PinHeader_2.54mm:PinHeader_1x08_P2.54mm_Vertical" (layer "F.Cu")
-    (at 115.05 47.3)
+    (at 115.04 47.28)
     (descr "Through hole straight pin header, 1x08, 2.54mm pitch, single row")
     (tags "Through hole pin header THT 1x08 2.54mm single row")
@@
     (property "Sheetname" "")
     (attr through_hole)
-    (fp_text reference "J3" (at 0 -2.33 unlocked) (layer "F.SilkS")
+    (fp_text reference "J3" (at 1.12 -2.35 unlocked) (layer "F.SilkS")
       (effects (font (size 0.7 0.7) (thickness 0.15)))
     )
@@
     (property "Sheetname" "")
     (attr through_hole)
-    (fp_text reference "J1" (at 8.265 3.85) (layer "F.SilkS")
+    (fp_text reference "J1" (at 8.7 3.76) (layer "F.SilkS")
       (effects (font (size 0.7 0.7) (thickness 0.15)))
     )
@@
     (property "Sheetname" "")
     (attr smd)
-    (fp_text reference "D2" (at 1.365 1.805 unlocked) (layer "F.SilkS")
+    (fp_text reference "D2" (at 1.32 2.06 unlocked) (layer "F.SilkS")
       (effects (font (size 0.7 0.7) (thickness 0.15)))
     )
@@
     (property "Sheetname" "")
     (attr smd)
-    (fp_text reference "R8" (at 0 1.65 270 unlocked) (layer "B.SilkS")
+    (fp_text reference "R8" (at 0.74 -2.1 unlocked) (layer "B.SilkS")
       (effects (font (size 0.7 0.7) (thickness 0.15)) (justify mirror))
     )
@@
     )
   )
+  (gr_line (start 117.51 41.08) (end 117.51 71.08) (layer "F.Cu") (width 0.2))
+  (gr_line (start 72.51 41.08) (end 117.51 41.08) (layer "F.Cu") (width 0.2))
+  (gr_line (start 117.51 71.08) (end 72.51 71.08) (layer "F.Cu") (width 0.2))
+  (gr_line (start 72.51 71.08) (end 72.51 41.08) (layer "F.Cu") (width 0.2))
+  (gr_line (start 72.51 71.08) (end 72.51 41.08) (layer "B.Cu") (width 0.2))
+  (gr_line (start 117.51 71.08) (end 72.51 71.08) (layer "B.Cu") (width 0.2))
+  (gr_line (start 72.51 41.08) (end 117.51 41.08) (layer "B.Cu") (width 0.2))
+  (gr_line (start 117.51 41.08) (end 117.51 71.08) (layer "B.Cu") (width 0.2))
   (gr_rect (start 72.5 41.07) (end 117.5 71.07) (layer "Edge.Cuts") (width 0.1) (fill none))
+  (gr_text "I+" (at 84.41 49.32) (layer "F.SilkS")
+    (effects (font (size 1 1) (thickness 0.15)))
+  )
+  (gr_text "Vcc" (at 106.94 46.29) (layer "F.SilkS")
+    (effects (font (size 0.7 0.7) (thickness 0.15)))
+  )
+  (gr_text "Vcc" (at 111.526667 62.03) (layer "F.SilkS")
+    (effects (font (size 0.7 0.7) (thickness 0.15)))
+  )
+  (gr_text "Is" (at 111.076667 63.19) (layer "F.SilkS")
+    (effects (font (size 0.7 0.7) (thickness 0.15)))
+  )
+  (gr_text "GND" (at 111.693333 65.51) (layer "F.SilkS")
+    (effects (font (size 0.7 0.7) (thickness 0.15)))
+  )
+  (gr_text "Isf" (at 111.276667 64.35) (layer "F.SilkS")
+    (effects (font (size 0.7 0.7) (thickness 0.15)))
+  )
+  (gr_text "Vdd" (at 111.41 46.28) (layer "F.SilkS")
+    (effects (font (size 0.7 0.7) (thickness 0.15)))
+  )
+  (gr_text "Vdd" (at 111.56 60.87) (layer "F.SilkS")
+    (effects (font (size 0.7 0.7) (thickness 0.15)))
+  )
+  (gr_text "Current sensor\nACS board\nv0.1" (at 93.42 66.64) (layer "F.SilkS")
+    (effects (font (size 0.7 0.7) (thickness 0.15)) (justify left))
+  )
+  (gr_text "GND" (at 111.693333 68.99) (layer "F.SilkS")
+    (effects (font (size 0.7 0.7) (thickness 0.15)))
+  )
+  (gr_text "I-" (at 84.29 63.15) (layer "F.SilkS")
+    (effects (font (size 1 1) (thickness 0.15)))
+  )
+  (gr_text "GND" (at 111.693333 67.83) (layer "F.SilkS")
+    (effects (font (size 0.7 0.7) (thickness 0.15)))
+  )
+  (gr_text "GND" (at 111.693333 66.67) (layer "F.SilkS")
+    (effects (font (size 0.7 0.7) (thickness 0.15)))
+  )
   (segment (start 92.075 52.2875) (end 92.1625 52.2) (width 0.5) (layer "F.Cu") (net 1))
   (segment (start 92.075 54.295) (end 92.075 52.2875) (width 0.5) (layer "F.Cu") (net 1))
@@
   )
   (zone (net 2) (net_name "GND") (layers F&B.Cu) (hatch edge 0.508)
-    (connect_pads (clearance 0.508))
+    (connect_pads (clearance 0.4))
     (min_thickness 0.508) (filled_areas_thickness no)
     (fill yes (thermal_gap 0.508) (thermal_bridge_width 0.508))
