File: buck-boost/buck-boost-xp.kicad_pcb (KiCad board)
At the start: 2 copper layers, 321.1 x 157.5 mm, 284 parts, among them J1 Conn_02x08_Odd_Even, J10 Conn_01x01, J11 Conn_01x02, J2 Conn_02x08_Odd_Even, J3 Conn_01x01, J4 Conn_01x01, J5 Conn_01x01, J6 Conn_01x01, J7 Conn_01x01, J8 Conn_01x01, J9 Conn_01x01, K1 Relay_SPDT, K2 Relay_SPDT, Q1 Q_NMOS_GDS, Q2 Q_NMOS_GDS, Q3 Q_NMOS_GDS, Q4 Q_NMOS_GDS, Q5 Q_NMOS_GDS, Q6 Q_NPN_BEC, Q7 Q_NPN_BEC, Q8 Q_NPN_BEC, Q9 Q_NPN_BEC, U1 1ED3125MU12F, U10 Opamp_Dual, U11 Opamp_Dual, U12 Opamp_Dual, U13 Opamp_Dual, U14 Opamp_Dual, U15 Opamp_Dual, U16 LMR33630ADDA, U18 LMR62014XMF_NOPB, U2 1ED3125MU12F, U3 ACS712ELCTR-20A, U4 TBA1-1212E, U5 TBA1-1212E, U6 1ED3125MU12F, U7 1ED3125MU12F, U8 ACS730xLCTR-20AB, U9 ACS712ELCTR-20A

Commit message: The recommendations discussed in the meeting must be implemented. The placement of some components must be improved.
Parts:
- D16: moved to B.Cu
- moved H4 235.8 mm to (64.8, 171.0)
- moved H3 162.9 mm to (47.2, 171.0)
- moved H2 152.0 mm to (56.8, 171.0)
- moved J8 116.4 mm to (259.8, 39.5)
- moved J7 115.2 mm to (279.8, 39.5)
- moved C65 113.6 mm to (100.8, 52.5)
- moved R92 113.6 mm to (98.2, 52.5)
- moved C63 113.6 mm to (101.4, 48.7)
- moved C64 113.6 mm to (100.5, 45.3)
- moved C101 113.5 mm to (78.8, 47.9)
- moved C102 113.5 mm to (83.0, 47.9)
- moved D17 113.5 mm to (71.7, 48.2)
- moved L3 113.5 mm to (93.0, 37.7)
- moved R93 113.5 mm to (95.2, 51.5)
- moved U16 113.5 mm to (93.6, 47.3)
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Routing:
- net /S3: track 64.4 -> 8.38 mm, vias 1 -> 0
- net /S4: track 59.7 -> 10.4 mm, vias 1 -> 0
- net /S1: track 54.1 -> 17.5 mm, vias 1 -> 0
- net /I_in_-: track 48.8 -> 79.1 mm
- net /S2: track 47.8 -> 19.5 mm, vias 1 -> 0
- net /Vs_S1: track 61.1 -> 32.8 mm, vias 24 -> 0
- net VDD: track 159.3 -> 131.3 mm, vias 6 -> 5
- net /IL-: track 64.8 -> 39.7 mm
- net /G_S4: track 27.6 -> 3.28 mm, vias 0 -> 1
- net /I_out_+: track 21.7 -> 44.6 mm
- net /Measurements/Current measurement/sig_cond_curr_sens3/out_: track 2.86 -> 23.0 mm
- net GND: track 167.6 -> 149.4 mm, vias 10 -> 22
- net /Drivers/Vcc_S3: track 35.9 -> 18.1 mm, vias 1 -> 0
- net /Measurements/Current measurement/I_out: track 4.20 -> 20.8 mm
- net /Drivers/Vcc_S1: track 36.0 -> 20.2 mm
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- added copper zone on B.Cu, net /IN+
- removed copper zone on B.Cu, net /I_in_+
- removed copper zone on B.Cu, net /I_in_-
- removed copper zone on F.Cu, net /I_out_+
- removed copper zone on F.Cu, net GND
- removed copper zone on F.Cu, net Net-(J3-Pin_1)
Other:
- board size 321.1 x 157.5 mm -> 265 x 132.8 mm

Commit message: V1.0 trying to improve the placement of the input relay
Parts:
- moved J7 61.3 mm to (279.5, 100.8), turned to 180 degrees
- moved C89 54.6 mm to (325.5, 56.9)
- moved R42 54.6 mm to (326.6, 67.5)
- moved R73 54.6 mm to (331.2, 51.8)
- moved R74 54.6 mm to (329.2, 51.8)
- moved R78 54.6 mm to (329.2, 56.0)
- moved C56 54.6 mm to (329.5, 68.5)
- moved C78 54.6 mm to (331.2, 56.0)
- moved C88 54.6 mm to (325.5, 54.9)
- moved R72 54.6 mm to (329.4, 66.5)
- moved R76 54.6 mm to (333.2, 56.0)
- moved U12 54.6 mm to (328.6, 61.7)
- moved C83 54.6 mm to (333.3, 61.0)
- moved R75 54.6 mm to (333.3, 64.5)
- moved R77 54.6 mm to (333.3, 59.0)
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Routing:
- net /I_out_+: track 44.6 -> 7.64 mm
- net /I_in_-: track 79.1 -> 52.2 mm
- net /K_in_A2: track 29.3 -> 8.20 mm
- net VDD: track 131.3 -> 120.1 mm
- removed copper zone on F.Cu, net /IL-
Other:
- board size 265 x 132.8 mm -> 265 x 120.2 mm

Commit message: Changing the position of the Gate drivers
Parts:
- C24, C25, C26, C27, C28, C29, L2, L4: moved to F.Cu
- moved H2 283.5 mm to (304.5, 31.8)
- moved H4 247.9 mm to (312.2, 157.5)
- moved H3 140.4 mm to (85.8, 33.5)
- moved K1 91.0 mm to (107.6, 147.0), turned to 90 degrees
- moved D13 87.6 mm to (107.6, 144.4), turned to 0 degrees
- moved J3 84.9 mm to (86.2, 103.8), turned to 90 degrees
- moved JP3 83.3 mm to (86.2, 118.8), turned to 180 degrees
- moved D14 82.8 mm to (106.6, 110.0)
- moved Q8 82.8 mm to (107.7, 107.2)
- moved R31 82.8 mm to (110.5, 104.4)
- moved R32 82.8 mm to (106.6, 104.4)
- moved R33 82.8 mm to (110.5, 110.0)
- moved JP2 80.0 mm to (102.5, 101.8), turned to 90 degrees
- moved JP4 77.8 mm to (196.8, 57.8), turned to -90 degrees
- moved C9 68.3 mm to (132.2, 130.2)
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Connections:
- J1 pad 1: /I_in_sens -> /V_dc_in_sens
- J1 pad 3: /IL_sens -> /I_in_sens
- J1 pad 5: /I_out_sens -> /IL_sens
- J1 pad 7: /V_dc_in_sens -> /V_dc_out_sens
- J1 pad 9: /V_dc_out_sens -> /I_out_sens
Routing:
- net /I_in_sens: track 1.99 -> 126.7 mm
- net /V_dc_in_sens: track 1.99 -> 108.8 mm
- net /V_out_sens: track 0.00 -> 103.2 mm
- net /V_dc_out_sens: track 2.00 -> 100.0 mm
- net VDD: track 120.1 -> 193.6 mm, vias 5 -> 2
- net /S3: track 8.38 -> 77.5 mm
- net /K_out: track 1.90 -> 51.9 mm
- net /S2: track 19.5 -> 65.6 mm
- net /S_load: track 1.98 -> 41.2 mm
- net /I_out_+: track 7.64 -> 46.3 mm
- net /I_in_-: track 52.2 -> 87.7 mm
- net /IL_sens: track 2.00 -> 31.4 mm
- net /Vs_S1: track 32.8 -> 54.0 mm, vias 0 -> 1
- net /Measurements/Current measurement/I_L: track 0.00 -> 20.1 mm
- net /S1: track 17.5 -> 0.00 mm
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- added copper zone on B.Cu, net /Vel
- added copper zone on F.Cu, net GND
- added copper zone on F.Cu, net Net-(D21-A)
- added copper zone on F.Cu, net Net-(J3-Pin_1)
- removed copper zone on B.Cu, net /IN+
Other:
- board size 265 x 120.2 mm -> 269 x 120 mm

Commit message: Update V1.0
Parts:
- C24, C25, C26, C27, C28, C29, L2, L4: moved to B.Cu
- moved J11 120.0 mm to (277.6, 53.8), turned to 180 degrees
- moved JP5 55.9 mm to (246.9, 58.2)
- moved JP4 47.0 mm to (243.7, 54.9), turned to 90 degrees
- moved R52 40.4 mm to (121.8, 53.0), turned to -90 degrees
- moved R53 40.4 mm to (126.3, 47.2), turned to -90 degrees
- moved C96 40.1 mm to (124.2, 47.2), turned to 90 degrees
- moved R54 39.3 mm to (121.8, 49.2)
- moved Q5 36.6 mm to (341.5, 70.5)
- moved R27 35.6 mm to (341.5, 66.2)
- moved R28 35.6 mm to (339.5, 66.2)
- moved JP1 35.6 mm to (341.8, 52.0)
- moved R30 35.6 mm to (339.4, 56.4)
- moved Q6 35.6 mm to (340.5, 61.3)
- moved Q7 35.6 mm to (336.9, 61.3)
- moved R29 35.6 mm to (337.4, 66.2)
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Connections:
- J1 pad 1: /V_dc_in_sens -> /I_in_sens
- J1 pad 11: /V_out_sens -> /V_dc_out_sens
- J1 pad 3: /I_in_sens -> /V_dc_in_sens
- J1 pad 7: /V_dc_out_sens -> /V_out_sens
Routing:
- net VDD: track 193.6 -> 487.1 mm, vias 2 -> 9
- net /K_in: track 10.6 -> 127.6 mm
- net /S1: track 0.00 -> 98.4 mm
- net VCC: track 24.8 -> 105.0 mm, vias 1 -> 2
- net /S4: track 0.00 -> 76.6 mm
- net /I_out_+: track 46.3 -> 107.1 mm, vias 0 -> 1
- net GND: track 151.2 -> 208.0 mm, vias 22 -> 32
- net /V_dc_out_sens: track 100.0 -> 44.8 mm
- net /V_out_sens: track 103.2 -> 51.0 mm
- net /IL-: track 34.9 -> 80.9 mm
- net /I_out_sens: track 2.00 -> 47.4 mm
- net /S_load: track 41.2 -> 1.98 mm
- net /S2: track 65.6 -> 102.8 mm, vias 0 -> 1
- net /K_in_A2: track 8.00 -> 42.1 mm, vias 0 -> 1
- net /G_S4: track 3.28 -> 35.8 mm
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- added copper zone on F.Cu, net /IL-
- added copper zone on F.Cu, net /I_out_+
- added copper zone on F.Cu, net /V_out
- added copper zone on B.Cu, net GND
- added copper zone on F.Cu, net Net-(U18-FB)
- added copper zone on F.Cu, net Net-(U18-/SHDN)
- added copper zone on B.Cu, net VCC
- added copper zone on F.Cu, net VCC
Other:
- board size 269 x 120 mm -> 268.5 x 118 mm

Commit message: Update V1.0
Parts:
- moved J11 185.2 mm to (92.5, 47.0), turned to 90 degrees
- moved H2 29.4 mm to (328.2, 49.0)
- moved H4 16.0 mm to (328.2, 157.8)
- moved TP1 4.00 mm to (144.0, 93.4)
- moved TP5 4.00 mm to (144.0, 89.8)
- moved JP5 1.80 mm to (248.7, 58.2)
- moved C1 1.65 mm to (156.3, 99.7)
- moved C4 1.65 mm to (156.3, 101.8)
- moved D2 1.65 mm to (143.6, 107.2)
- moved D3 1.65 mm to (146.2, 102.0)
- moved R3 1.65 mm to (156.3, 97.5)
- moved C2 1.65 mm to (160.5, 107.3)
- moved C3 1.65 mm to (160.5, 101.2)
- moved C5 1.65 mm to (149.4, 97.5)
- moved C6 1.65 mm to (149.4, 99.7)
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Routing:
- net VDD: track 487.1 -> 773.1 mm, vias 9 -> 19
- net VCC: track 105.0 -> 308.6 mm, vias 2 -> 4
- net /V_out_sens: track 51.0 -> 149.3 mm
- net /S_load: track 1.98 -> 96.3 mm, vias 0 -> 1
- net /I_out_sens: track 47.4 -> 132.8 mm
- net /V_dc_out_sens: track 44.8 -> 115.7 mm
- net /K_out: track 30.3 -> 78.6 mm
- net GND: track 208.0 -> 242.7 mm, vias 32 -> 37
- net /IL_sens: track 13.2 -> 41.3 mm, vias 0 -> 2
- net /G_S2: track 19.0 -> 41.6 mm
- net Net-(J2-Pin_11): track 0.00 -> 21.5 mm
- net Net-(JP1-A): track 0.00 -> 20.2 mm
- net /G_S1: track 35.8 -> 42.9 mm
- net /G_S_load: track 0.00 -> 6.80 mm
- net /K_in: track 127.6 -> 134.4 mm
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- added copper zone on F.Cu, net /buck_boost_power_stage/Load-
- removed copper zone on B.Cu, net VCC
Other:
- outline, holes or cut-outs redrawn

Commit message: Update V1.0
Parts:
- D1, D10, D11, D2, D4, D7: moved to B.Cu
- moved TP1 15.0 mm to (138.8, 107.5)
- moved TP5 15.0 mm to (138.8, 103.9)
- moved TP4 14.3 mm to (226.5, 107.5)
- moved TP8 14.3 mm to (226.5, 103.9)
- moved D7 7.01 mm to (280.3, 100.6), turned to -90 degrees
- moved D4 7.01 mm to (190.9, 100.6), turned to -90 degrees
- moved R4 4.81 mm to (145.8, 105.5), turned to 90 degrees
- moved R20 4.79 mm to (233.6, 105.5), turned to 90 degrees
- moved R5 4.69 mm to (142.6, 105.5), turned to 90 degrees
- moved R21 4.68 mm to (230.3, 105.5), turned to 90 degrees
- moved TP2 3.62 mm to (196.8, 106.5)
- moved TP6 3.62 mm to (196.8, 102.9)
- moved D10 2.78 mm to (233.7, 99.7), turned to -90 degrees
- moved D12 2.53 mm to (231.9, 100.5), turned to 180 degrees
- moved D3 2.53 mm to (144.2, 100.5), turned to 180 degrees
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Routing:
- net /K_in: track 134.4 -> 200.6 mm, vias 0 -> 1
- net /K_out: track 78.6 -> 135.1 mm, vias 0 -> 2
- net GND: track 242.7 -> 195.1 mm, vias 37 -> 39
- net Net-(J2-Pin_6): track 0.00 -> 31.5 mm
- net /G_S1: track 42.9 -> 21.5 mm
- net /G_S4: track 40.8 -> 22.3 mm
- net /Vs_S1: track 73.2 -> 84.5 mm
- net /IL-: track 80.9 -> 70.6 mm, vias 0 -> 1
- net Net-(D10-A): track 18.4 -> 11.9 mm, vias 0 -> 1
- net /Drivers/Vcc_S3: track 35.2 -> 41.2 mm
- net /Drivers/Vcc_S1: track 22.0 -> 27.9 mm
- net Net-(D1-A): track 18.4 -> 13.1 mm, vias 0 -> 1
- net Net-(J2-Pin_11): track 21.5 -> 22.9 mm
- net /I_in_sens: track 105.0 -> 103.6 mm
- net /I_in_-: track 83.3 -> 82.3 mm
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