File: buck-boost/buck-boost-xp.kicad_pcb (KiCad board)
At the start: 2 copper layers, 268.5 x 118 mm, 284 parts, among them J1 Conn_02x08_Odd_Even, J10 Conn_01x01, J11 Conn_01x02, J2 Conn_02x08_Odd_Even, J3 Conn_01x01, J4 Conn_01x01, J5 Conn_01x01, J6 Conn_01x01, J7 Conn_01x01, J8 Conn_01x01, J9 Conn_01x01, K1 Relay_SPDT, K2 Relay_SPDT, Q1 Q_NMOS_GDS, Q2 Q_NMOS_GDS, Q3 Q_NMOS_GDS, Q4 Q_NMOS_GDS, Q5 Q_NMOS_GDS, Q6 Q_NPN_BEC, Q7 Q_NPN_BEC, Q8 Q_NPN_BEC, Q9 Q_NPN_BEC, U1 1ED3125MU12F, U10 Opamp_Dual, U11 Opamp_Dual, U12 Opamp_Dual, U13 Opamp_Dual, U14 Opamp_Dual, U15 Opamp_Dual, U16 LMR33630ADDA, U18 LMR62014XMF_NOPB, U2 1ED3125MU12F, U3 ACS712ELCTR-20A, U4 TBA1-1212E, U5 TBA1-1212E, U6 1ED3125MU12F, U7 1ED3125MU12F, U8 ACS730xLCTR-20AB, U9 ACS712ELCTR-20A

Commit message: V1.0 finished. Teardrops were added.
Parts:
- added H5: MountingHole, MountingHole:MountingHole_3.2mm_M3, F.Cu at (202.2, 157.8)
- added H6: MountingHole, MountingHole:MountingHole_3.2mm_M3, F.Cu at (202.2, 67.0)
- moved JP5 2.25 mm to (248.7, 60.5)
- moved R88 0.60 mm to (108.0, 66.9)
- moved Q7 0.42 mm to (336.5, 61.3)
Routing:
- net GND: track 195.1 -> 22.8 mm, vias 39 -> 33
- net VDD: track 772.3 -> 749.6 mm, vias 19 -> 18
- net /S4: track 76.6 -> 83.0 mm
- net /S3: track 87.8 -> 93.9 mm
- net /S1: track 96.7 -> 102.4 mm
- net /S2: track 102.0 -> 107.3 mm
- net /S_load: track 96.3 -> 98.5 mm
- net /K_in: track 200.6 -> 199.1 mm
- net /G_S4: track 22.3 -> 20.9 mm
- net /V_out: track 19.6 -> 18.3 mm
- net Net-(J2-Pin_6): track 31.5 -> 32.4 mm
- net /G_S1: track 21.5 -> 20.5 mm
- net /IL_sens: track 41.3 -> 42.2 mm, vias 2 -> 1
- net /I_out_+: track 107.1 -> 108.0 mm
- net Net-(U13B-+): track 3.72 -> 3.01 mm
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Other:
- outline, holes or cut-outs redrawn
- board text added: "IN+"
- board text added: "IN-"
- board text added: "LOAD+"
- board text added: "LOAD-"
- board text added: "OUT+"
- board text added: "OUT-"
- board text added: "Vaux+"
- board text added: "Vaux-"

Commit message: Updated V1.0. Some changes regarding review. 16.12.2024 still to be done
Parts:
- moved H6 104.2 mm to (98.0, 66.5)
- moved C14 103.5 mm to (79.0, 144.2), turned to 0 degrees
- moved C16 82.5 mm to (202.8, 144.2)
- moved J1 77.0 mm to (114.0, 51.5)
- moved C9 66.4 mm to (66.3, 137.5), turned to 90 degrees
- moved TP1 66.0 mm to (72.9, 106.4)
- moved TP5 66.0 mm to (72.9, 102.7)
- moved R6 66.0 mm to (36.5, 116.5)
- moved C8 66.0 mm to (66.3, 149.3)
- moved C30 66.0 mm to (199.1, 99.7)
- moved C34 66.0 mm to (206.0, 101.8)
- moved C35 66.0 mm to (206.0, 99.7)
- moved C36 66.0 mm to (206.0, 97.5)
- moved C48 66.0 mm to (231.3, 107.9)
- moved C49 66.0 mm to (231.3, 105.8)
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Routing:
- net /K_out: track 135.1 -> 32.5 mm, vias 2 -> 0
- net /S_load: track 98.5 -> 1.98 mm, vias 1 -> 0
- net /K_in: track 199.1 -> 143.1 mm
- net /I_out_+: track 108.0 -> 64.2 mm, vias 1 -> 2
- net Net-(J2-Pin_6): track 32.4 -> 0.00 mm
- net /I_in_-: track 82.3 -> 52.1 mm, vias 0 -> 1
- net /V_out_sens: track 149.0 -> 176.4 mm
- net /V_dc_out_sens: track 116.0 -> 141.6 mm
- net /I_out_sens: track 132.9 -> 158.3 mm
- net Net-(J2-Pin_11): track 22.9 -> 0.00 mm
- net VDD: track 749.6 -> 770.2 mm
- net /IL_sens: track 42.2 -> 60.5 mm, vias 1 -> 2
- net GND: track 22.8 -> 11.0 mm, vias 33 -> 35
- net /S4: track 83.0 -> 72.0 mm
- net /S3: track 93.9 -> 83.1 mm
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- added copper zone on B.Cu, net /IN+
- added copper zone on B.Cu, net /V_out
Other:
- outline, holes or cut-outs redrawn
- board text added: "+"
- board text added: "-"
- board text added: "5V"

Commit message: V1.1. Changes regarding to Review 16.12.2024
Parts:
- added H7: MountingHole, MountingHole:MountingHole_3.2mm_M3, F.Cu at (210.8, 66.5)
- moved JP5 14.3 mm to (207.7, 46.9)
- moved JP4 6.23 mm to (196.1, 47.0)
- moved H2 2.75 mm to (265.0, 49.0)
- moved TP4 1.13 mm to (160.6, 106.4)
- moved TP8 1.13 mm to (160.6, 102.7)
- moved C90 0.25 mm to (66.5, 48.2)
- moved C97 0.25 mm to (66.5, 51.5)
- moved TP2 0.14 mm to (130.9, 106.4)
Routing:
- net /K_out: track 32.5 -> 124.4 mm, vias 0 -> 6
- net /S_load: track 1.98 -> 80.8 mm
- net /K_in: track 143.1 -> 216.4 mm, vias 1 -> 0
- net Net-(J2-Pin_6): track 0.00 -> 44.1 mm, vias 0 -> 1
- net Net-(J2-Pin_11): track 0.00 -> 26.9 mm
- net GND: track 11.0 -> 15.3 mm, vias 35 -> 44
- net /G_S4: track 20.9 -> 22.8 mm
- net /I_in_sens: track 99.6 -> 98.4 mm
- net /V_dc_out_sens: track 141.6 -> 140.6 mm
- net /V_dc_in_sens: track 84.5 -> 83.9 mm
- net VDD: track 770.2 -> 770.8 mm, vias 18 -> 17
- net /S2: track 113.3 -> 112.7 mm
- net /I_out_sens: track 158.3 -> 157.8 mm

Commit message: V1.2. New relay foot print added with 3D figure
Parts:
- K1, K2: footprint Relay_THT:Relay_SPDT_RAYEX-L90S -> CL_Relay:T9GV5L14-5
- moved K1 17.7 mm to (32.8, 131.6), turned to 0 degrees
- moved K2 17.3 mm to (258.1, 128.2), turned to 180 degrees
- moved JP4 12.7 mm to (204.2, 56.8)
- moved JP5 6.21 mm to (207.9, 53.1)
- moved D16 0.46 mm to (249.4, 115.4)
- moved TP2 0.18 mm to (130.9, 106.5)
Routing:
- net /I_in_-: track 52.1 -> 85.2 mm
- net /I_out_+: track 64.2 -> 96.3 mm
- net Net-(J2-Pin_11): track 26.9 -> 39.6 mm, vias 0 -> 2
- net /K_in: track 216.4 -> 228.9 mm, vias 0 -> 1
- net /S_load: track 80.8 -> 72.7 mm, vias 0 -> 2
- net /V_dc_out_sens: track 140.6 -> 132.8 mm, vias 0 -> 4
- net Net-(J2-Pin_6): track 44.1 -> 40.3 mm, vias 1 -> 0
- net VDD: track 770.8 -> 772.3 mm
- net VCC: track 308.9 -> 309.7 mm
- net /IL_sens: track 60.5 -> 61.2 mm
- net /K_out: track 124.4 -> 124.8 mm, vias 6 -> 4
