File: buck-boost/gd_1ed3125mu12f.kicad_sch (KiCad schematic)
At the start: 20 parts, among them U1 1ED3125MU12F

Commit message: Update V1.0
Other:
- note removed: "WHy MELF footprint ? SEE https://www.infineon.com/dgdl/Infineon-EVAL-1ED3122Mx12H-ApplicationNotes-v01_10-EN.pdf?fileId=5546d46274f6cd4c0174f821f169026f"
Changed lines of the file:
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@@
-		)
-	)
-	(text "WHy MELF footprint ? SEE https://www.infineon.com/dgdl/Infineon-EVAL-1ED3122Mx12H-ApplicationNotes-v01_10-EN.pdf?fileId=5546d46274f6cd4c0174f821f169026f\n"
-		(exclude_from_sim no)
-		(at 180.848 62.484 0)
-		(effects
-			(font
-				(size 1.27 1.27)
-			)
 		)
 	)
