File: buck-boost/buck_boost_power_stage.kicad_sch (KiCad schematic)
At the start: 27 parts, among them K1 Relay_SPDT, K2 Relay_SPDT, Q1 Q_NMOS_GDS, Q2 Q_NMOS_GDS, Q3 Q_NMOS_GDS, Q4 Q_NMOS_GDS, Q5 Q_NMOS_GDS

Commit message: V1.2. New relay foot print added with 3D figure
Parts:
- K1, K2: footprint Relay_THT:Relay_SPDT_RAYEX-L90S -> CL_Relay:T9GV5L14-5
Changed lines of the file:
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@@
 			)
 		)
-		(property "Footprint" "Relay_THT:Relay_SPDT_RAYEX-L90S"
+		(property "Footprint" "CL_Relay:T9GV5L14-5"
 			(at 231.14 41.91 0)
 			(effects
@@
 			)
 		)
-		(property "Footprint" "Relay_THT:Relay_SPDT_RAYEX-L90S"
+		(property "Footprint" "CL_Relay:T9GV5L14-5"
 			(at 40.64 41.91 0)
 			(effects
